File: ai-camera-rev3.1/ai-camera-rev3.1.kicad_pcb (KiCad board)
At the start: 4 copper layers, 70 x 70 mm, 178 parts, among them J1 Conn-01x02_P2mm_NONAME_JST-PH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, J2 TYPE-C-31-M-12, J3 MAXLAB, J4 Conn-02x10_P2.54mm_B-2100S20P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, J5 Conn-01x02_P1.25mm_10114829-1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, J6 Conn_01x24_FFC_0.5mm_AFC01-S2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, Q1 2N7002, Q10 2N7002, Q2 2N7002, Q3 AO3401A, Q4 AO3401A, Q5 2N7002, Q6 AO3401A, Q7 2N7002, Q8 AO3401A, Q9 2N7002, SW1 SW_PB_90deg_K2-1102AQ-H4CW-01, SW2 SW_PB_TS-1187A-B-A-B, SW3 SW_PB_TS-1187A-B-A-B, SW4 SW_PB_90deg_K2-1102AQ-H4CW-01, U1 TP4057-42-SOT26-R, U10 ESP32-S3-WROOM-1-N16R8, U11 MT9284-28J, U12 LTR-303ALS-01, U2 XC6206-2.8V, U3 PCF85063AT, U4 TI_SN74LVC1G373DBVR, U5 SY8089AAAC, U6 PIR_AS312, U7 XC6206-2.8V, U8 RT9166-12GVL, U9 AP1511B, Y1 32.768kHz_Q13FC1350000400

Commit message: rev3.1: fab files ready to be released
Changed lines of the file:
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@@
       (drillshape 0)
       (scaleselection 1)
-      (outputdirectory "fab/jlcpcb/gerbs/")
+      (outputdirectory "fab/fabpcb/gerbs/")
     )
   )
@@
     (fp_line (start 1.75 1.4) (end 1.75 -1.4)
       (stroke (width 0.1) (type solid)) (layer "F.Fab"))
-    (pad "1" smd roundrect (at -1.5375 0 180) (size 1.325 2.35) (layers "F.Cu" "F.Paste" "F.Mask") (roundrect_rratio 0.188679)
+    (pad "1" smd roundrect (at -1.5375 0 180) (size 1.325 2.35) (layers "F.Cu" "F.Paste" "F.Mask") (roundrect_rratio 0.1886792453)
       (net 4 "+BATT") (pintype "passive"))
-    (pad "2" smd roundrect (at 1.5375 0 180) (size 1.325 2.35) (layers "F.Cu" "F.Paste" "F.Mask") (roundrect_rratio 0.188679)
+    (pad "2" smd roundrect (at 1.5375 0 180) (size 1.325 2.35) (layers "F.Cu" "F.Paste" "F.Mask") (roundrect_rratio 0.1886792453)
       (net 1 "GND") (pintype "passive"))
     (model "${KICAD6_3DMODEL_DIR}/Capacitor_Tantalum_SMD.3dshapes/CP_EIA-3528-15_AVX-H.wrl"
@@
     (fp_line (start 1.75 1.4) (end 1.75 -1.4)
       (stroke (width 0.1) (type solid)) (layer "F.Fab"))
-    (pad "1" smd roundrect (at -1.5375 0 180) (size 1.325 2.35) (layers "F.Cu" "F.Paste" "F.Mask") (roundrect_rratio 0.188679)
+    (pad "1" smd roundrect (at -1.5375 0 180) (size 1.325 2.35) (layers "F.Cu" "F.Paste" "F.Mask") (roundrect_rratio 0.1886792453)
       (net 97 "Net-(Q6-S)") (pintype "passive"))
-    (pad "2" smd roundrect (at 1.5375 0 180) (size 1.325 2.35) (layers "F.Cu" "F.Paste" "F.Mask") (roundrect_rratio 0.188679)
+    (pad "2" smd roundrect (at 1.5375 0 180) (size 1.325 2.35) (layers "F.Cu" "F.Paste" "F.Mask") (roundrect_rratio 0.1886792453)
       (net 1 "GND") (pintype "passive"))
     (model "${KICAD6_3DMODEL_DIR}/Capacitor_Tantalum_SMD.3dshapes/CP_EIA-3528-15_AVX-H.wrl"
@@
     (fp_line (start 1.75 1.4) (end 1.75 -1.4)
       (stroke (width 0.1) (type solid)) (layer "F.Fab"))
-    (pad "1" smd roundrect (at -1.5375 0 90) (size 1.325 2.35) (layers "F.Cu" "F.Paste" "F.Mask") (roundrect_rratio 0.188679)
+    (pad "1" smd roundrect (at -1.5375 0 90) (size 1.325 2.35) (layers "F.Cu" "F.Paste" "F.Mask") (roundrect_rratio 0.1886792453)
       (net 6 "+3V3") (pintype "passive"))
-    (pad "2" smd roundrect (at 1.5375 0 90) (size 1.325 2.35) (layers "F.Cu" "F.Paste" "F.Mask") (roundrect_rratio 0.188679)
+    (pad "2" smd roundrect (at 1.5375 0 90) (size 1.325 2.35) (layers "F.Cu" "F.Paste" "F.Mask") (roundrect_rratio 0.1886792453)
       (net 1 "GND") (pintype "passive"))
     (model "${KICAD6_3DMODEL_DIR}/Capacitor_Tantalum_SMD.3dshapes/CP_EIA-3528-15_AVX-H.wrl"
@@
     (fp_line (start 1.75 1.4) (end 1.75 -1.4)
       (stroke (width 0.1) (type solid)) (layer "F.Fab"))
-    (pad "1" smd roundrect (at -1.5375 0 180) (size 1.325 2.35) (layers "F.Cu" "F.Paste" "F.Mask") (roundrect_rratio 0.188679)
+    (pad "1" smd roundrect (at -1.5375 0 180) (size 1.325 2.35) (layers "F.Cu" "F.Paste" "F.Mask") (roundrect_rratio 0.1886792453)
       (net 97 "Net-(Q6-S)") (pintype "passive"))
-    (pad "2" smd roundrect (at 1.5375 0 180) (size 1.325 2.35) (layers "F.Cu" "F.Paste" "F.Mask") (roundrect_rratio 0.188679)
+    (pad "2" smd roundrect (at 1.5375 0 180) (size 1.325 2.35) (layers "F.Cu" "F.Paste" "F.Mask") (roundrect_rratio 0.1886792453)
       (net 1 "GND") (pintype "passive"))
     (model "${KICAD6_3DMODEL_DIR}/Capacitor_Tantalum_SMD.3dshapes/CP_EIA-3528-15_AVX-H.wrl"
@@
     (fp_line (start 1.75 1.4) (end -1.05 1.4)
       (stroke (width 0.1) (type solid)) (layer "B.Fab"))
-    (pad "1" smd roundrect (at -1.5375 0 180) (size 1.325 2.35) (layers "B.Cu" "B.Paste" "B.Mask") (roundrect_rratio 0.188679)
+    (pad "1" smd roundrect (at -1.5375 0 180) (size 1.325 2.35) (layers "B.Cu" "B.Paste" "B.Mask") (roundrect_rratio 0.1886792453)
       (net 6 "+3V3") (pintype "passive"))
-    (pad "2" smd roundrect (at 1.5375 0 180) (size 1.325 2.35) (layers "B.Cu" "B.Paste" "B.Mask") (roundrect_rratio 0.188679)
+    (pad "2" smd roundrect (at 1.5375 0 180) (size 1.325 2.35) (layers "B.Cu" "B.Paste" "B.Mask") (roundrect_rratio 0.1886792453)
       (net 1 "GND") (pintype "passive"))
     (model "${KICAD6_3DMODEL_DIR}/Capacitor_Tantalum_SMD.3dshapes/CP_EIA-3528-15_AVX-H.wrl"
@@
     (fp_line (start 1.75 1.4) (end -1.05 1.4)
       (stroke (width 0.1) (type solid)) (layer "B.Fab"))
-    (pad "1" smd roundrect (at -1.5375 0 180) (size 1.325 2.35) (layers "B.Cu" "B.Paste" "B.Mask") (roundrect_rratio 0.188679)
+    (pad "1" smd roundrect (at -1.5375 0 180) (size 1.325 2.35) (layers "B.Cu" "B.Paste" "B.Mask") (roundrect_rratio 0.1886792453)
       (net 6 "+3V3") (pintype "passive"))
-    (pad "2" smd roundrect (at 1.5375 0 180) (size 1.325 2.35) (layers "B.Cu" "B.Paste" "B.Mask") (roundrect_rratio 0.188679)
+    (pad "2" smd roundrect (at 1.5375 0 180) (size 1.325 2.35) (layers "B.Cu" "B.Paste" "B.Mask") (roundrect_rratio 0.1886792453)
       (net 1 "GND") (pintype "passive"))
     (model "${KICAD6_3DMODEL_DIR}/Capacitor_Tantalum_SMD.3dshapes/CP_EIA-3528-15_AVX-H.wrl"
@@
     (fp_line (start 1.75 1.4) (end -1.05 1.4)
       (stroke (width 0.1) (type solid)) (layer "B.Fab"))
-    (pad "1" smd roundrect (at -1.5375 0 180) (size 1.325 2.35) (layers "B.Cu" "B.Paste" "B.Mask") (roundrect_rratio 0.188679)
+    (pad "1" smd roundrect (at -1.5375 0 180) (size 1.325 2.35) (layers "B.Cu" "B.Paste" "B.Mask") (roundrect_rratio 0.1886792453)
       (net 6 "+3V3") (pintype "passive"))
-    (pad "2" smd roundrect (at 1.5375 0 180) (size 1.325 2.35) (layers "B.Cu" "B.Paste" "B.Mask") (roundrect_rratio 0.188679)
+    (pad "2" smd roundrect (at 1.5375 0 180) (size 1.325 2.35) (layers "B.Cu" "B.Paste" "B.Mask") (roundrect_rratio 0.1886792453)
       (net 1 "GND") (pintype "passive"))
     (model "${KICAD6_3DMODEL_DIR}/Capacitor_Tantalum_SMD.3dshapes/CP_EIA-3528-15_AVX-H.wrl"
